Commit message: Migration in progress

File: morpheus_description/urdf/macros/ur5e_macro.xacro (robot description, xacro)
@@ -4,33 +4,31 @@
 <robot name="ur5e" xmlns:xacro="http://www.ros.org/wiki/xacro">
   <xacro:macro name="ur5e" params="
-    prefix
+    name:='ur5e'
+    tf_prefix
     parent
-    transmission_hw_interface:=hardware_interface/PositionJointInterface
     joint_limits_parameters_file:='$(find ur_description)/config/ur5e/joint_limits.yaml'
     tcp_offset
     *origin">
     <!-- ur5e -->
-    <xacro:include filename="$(find ur_description)/urdf/inc/ur_macro.xacro" />
+    <xacro:include filename="$(find ur_description)/urdf/ur_macro.xacro" />
     <xacro:ur_robot
-      prefix="${prefix}"
+      name="${name}"
+      tf_prefix="${tf_prefix}"
+      parent="${parent}"
       joint_limits_parameters_file="${joint_limits_parameters_file}"
       kinematics_parameters_file='$(find ur_description)/config/ur5e/default_kinematics.yaml'
       physical_parameters_file='$(find ur_description)/config/ur5e/physical_parameters.yaml'
       visual_parameters_file='$(find ur_description)/config/ur5e/visual_parameters.yaml'
-      transmission_hw_interface="${transmission_hw_interface}"
       safety_limits="false"
       safety_pos_margin="0.15"
       safety_k_position="20"
-    />
-    <joint name="${prefix}ur5e_base_joint" type="fixed">
-      <parent link="${parent}" />
-      <child link="${prefix}base_link" />
+      >
       <xacro:insert_block name="origin" />
-    </joint>
+    </xacro:ur_robot>
     <!-- Add an additional link to plan with. Oriented like the Trossen ee_gripper_link frame. -->
-    <link name="${prefix}tcp_link" />
-    <joint name="${prefix}tcp_joint" type="fixed">
-      <parent link="${prefix}wrist_3_link" />
-      <child link="${prefix}tcp_link" />
+    <link name="${tf_prefix}tcp_link" />
+    <joint name="${tf_prefix}tcp_joint" type="fixed">
+      <parent link="${tf_prefix}wrist_3_link" />
+      <child link="${tf_prefix}tcp_link" />
       <origin rpy="0 ${-pi/2} ${-pi/2}" xyz="0 0 ${tcp_offset}" />
     </joint>
