Commit message: Dockerfile and compose rework for GPU, Gazebo works but GPU passthrough does not.

File: morpheus_description/urdf/macros/Test_Block_1.xacro (robot description, xacro)
@@ -12,5 +12,5 @@
             <origin rpy="0 0 0" xyz="0 0 0"/>
             <geometry>
-                <mesh filename="package://morpheus_description/meshes/components/visual/test_block_1.stl" scale="${scale} ${scale} ${scale}"/>
+                <mesh filename="file://$(find morpheus_description)/meshes/components/visual/test_block_1.stl" scale="${scale} ${scale} ${scale}"/>
             </geometry>
             <material name="grey">
@@ -21,5 +21,5 @@
             <origin rpy="0 0 0" xyz="0 0 0" />
             <geometry>
-                <mesh filename="package://morpheus_description/meshes/components/collision/test_block_1.stl" scale="${scale} ${scale} ${scale}"/>
+                <mesh filename="file://$(find morpheus_description)/meshes/components/collision/test_block_1.stl" scale="${scale} ${scale} ${scale}"/>
             </geometry>
         </collision>

File: morpheus_description/urdf/macros/a_bot_macro.xacro (robot description, xacro)
@@ -8,13 +8,9 @@
         prefix
         parent
-        transmission_hw_interface:=hardware_interface/PositionJointInterface
-        joint_limits_parameters_file:='$(find ur_description)/config/ur5e/joint_limits.yaml'
         *origin">
         <xacro:ur5e
-            prefix="${prefix}"
+            tf_prefix="${prefix}"
             parent="${parent}"
             tcp_offset="0.163"
-            joint_limits_parameters_file="${joint_limits_parameters_file}"
-            transmission_hw_interface="${transmission_hw_interface}"
         >
             <xacro:insert_block name="origin" />
@@ -29,5 +25,5 @@
             prefix="${prefix}"
             parent="${prefix}d415_mount_attach_link"
-            transmission_hw_interface="${transmission_hw_interface}"
+            transmission_hw_interface="hardware_interface/PositionJointInterface"
             add_cable_protector="true"
         >

File: morpheus_description/urdf/macros/b_bot_macro.xacro (robot description, xacro)
@@ -8,13 +8,9 @@
         prefix
         parent
-        transmission_hw_interface:=hardware_interface/PositionJointInterface
-        joint_limits_parameters_file:='$(find ur_description)/config/ur5e/joint_limits.yaml'
         *origin">
         <xacro:ur5e
-            prefix="${prefix}"
+            tf_prefix="${prefix}"
             parent="${parent}"
             tcp_offset="0.223"
-            joint_limits_parameters_file="${joint_limits_parameters_file}"
-            transmission_hw_interface="${transmission_hw_interface}"
         >
             <xacro:insert_block name="origin" />
@@ -29,5 +25,5 @@
             prefix="${prefix}"
             parent="${prefix}d415_mount_attach_link"
-            hw_interface="${transmission_hw_interface}"
+            hw_interface="hardware_interface/PositionJointInterface"
         >
             <origin xyz="0 0 0.0026" rpy="0 0 ${pi}" />

File: morpheus_description/urdf/macros/bar_12in.xacro (robot description, xacro)
@@ -12,5 +12,5 @@
             <origin rpy="0 0 0" xyz="0 0 0"/>
             <geometry>
-                <mesh filename="package://morpheus_description/meshes/components/visual/bar_12in.obj" scale="${scale} ${scale} ${scale}"/>
+                <mesh filename="file://$(find morpheus_description)/meshes/components/visual/bar_12in.obj" scale="${scale} ${scale} ${scale}"/>
             </geometry>
             <material name="grey">
@@ -21,5 +21,5 @@
             <origin rpy="0 0 0" xyz="0 0 0" />
             <geometry>
-                <mesh filename="package://morpheus_description/meshes/components/collision/bar_12in.obj" scale="${scale} ${scale} ${scale}"/>
+                <mesh filename="file://$(find morpheus_description)/meshes/components/collision/bar_12in.obj" scale="${scale} ${scale} ${scale}"/>
             </geometry>
         </collision>

File: morpheus_description/urdf/macros/bar_4in.xacro (robot description, xacro)
@@ -12,5 +12,5 @@
             <origin rpy="1.57079632679 0 0" xyz="0 ${scale * 1} 0"/>
             <geometry>
-                <mesh filename="package://morpheus_description/meshes/components/visual/bar_4in.obj" scale="${scale} ${scale} ${scale}"/>
+                <mesh filename="file://$(find morpheus_description)/meshes/components/visual/bar_4in.obj" scale="${scale} ${scale} ${scale}"/>
             </geometry>
             <material name="grey">
@@ -21,5 +21,5 @@
             <origin rpy="1.57079632679 0 0" xyz="0 ${scale * 1} 0" />
             <geometry>
-                <mesh filename="package://morpheus_description/meshes/components/collision/bar_4in.obj" scale="${scale} ${scale} ${scale}"/>
+                <mesh filename="file://$(find morpheus_description)/meshes/components/collision/bar_4in.obj" scale="${scale} ${scale} ${scale}"/>
             </geometry>
         </collision>

File: morpheus_description/urdf/macros/block.xacro (robot description, xacro)
@@ -12,5 +12,5 @@
             <origin rpy="1.57079632679 0 0" xyz="0 0 0"/>
             <geometry>
-                <mesh filename="package://morpheus_description/meshes/components/visual/block.obj" scale="${scale} ${scale} ${scale}"/>
+                <mesh filename="file://$(find morpheus_description)/meshes/components/visual/block.obj" scale="${scale} ${scale} ${scale}"/>
             </geometry>
             <material name="grey">
@@ -21,5 +21,5 @@
             <origin rpy="1.57079632679 0 0" xyz="0 0 0" />
             <geometry>
-                <mesh filename="package://morpheus_description/meshes/components/collision/block.obj" scale="${scale} ${scale} ${scale}"/>
+                <mesh filename="file://$(find morpheus_description)/meshes/components/collision/block.obj" scale="${scale} ${scale} ${scale}"/>
             </geometry>
         </collision>

File: morpheus_description/urdf/macros/d415_mount_macro.xacro (robot description, xacro)
@@ -15,5 +15,5 @@
                 <geometry>
                     <mesh
-                        filename="package://homestri_description/meshes/visual/d415_mount.stl"
+                        filename="file://$(find morpheus_description)/meshes/visual/d415_mount.stl"
                         scale="0.001 0.001 0.001" />
                 </geometry>
@@ -26,5 +26,5 @@
                 <geometry>
                     <mesh
-                        filename="package://homestri_description/meshes/collision/d415_mount.stl"
+                        filename="file://$(find morpheus_description)/meshes/collision/d415_mount.stl"
                         scale="0.001 0.001 0.001" />
                 </geometry>

File: morpheus_description/urdf/macros/dragon_simple.xacro (robot description, xacro)
@@ -12,5 +12,5 @@
             <origin rpy="1.57079632679 0 0" xyz="0 0 0"/>
             <geometry>
-                <mesh filename="package://morpheus_description/meshes/components/visual/dragon_simple.obj" scale="${scale} ${scale} ${scale}"/>
+                <mesh filename="file://$(find morpheus_description)/meshes/components/visual/dragon_simple.obj" scale="${scale} ${scale} ${scale}"/>
             </geometry>
             <material name="grey">
@@ -21,5 +21,5 @@
             <origin rpy="1.57079632679 0 0" xyz="0 0 0" />
             <geometry>
-                <mesh filename="package://morpheus_description/meshes/components/collision/dragon_simple.obj" scale="${scale} ${scale} ${scale}"/>
+                <mesh filename="file://$(find morpheus_description)/meshes/components/collision/dragon_simple.obj" scale="${scale} ${scale} ${scale}"/>
             </geometry>
         </collision>

File: morpheus_description/urdf/macros/foam.xacro (robot description, xacro)
@@ -12,5 +12,5 @@
             <origin rpy="1.57079632679 0 0" xyz="0 0 0"/>
             <geometry>
-                <mesh filename="package://morpheus_description/meshes/components/visual/foam.obj" scale="${scale} ${scale} ${scale}"/>
+                <mesh filename="file://$(find morpheus_description)/meshes/components/visual/foam.obj" scale="${scale} ${scale} ${scale}"/>
             </geometry>
             <material name="grey">
@@ -21,5 +21,5 @@
             <origin rpy="1.57079632679 0 0" xyz="0 0 0" />
             <geometry>
-                <mesh filename="package://morpheus_description/meshes/components/collision/foam.obj" scale="${scale} ${scale} ${scale}"/>
+                <mesh filename="file://$(find morpheus_description)/meshes/components/collision/foam.obj" scale="${scale} ${scale} ${scale}"/>
             </geometry>
         </collision>

File: morpheus_description/urdf/macros/hera_obstacle_course_mesh.xacro (robot description, xacro)
@@ -8,5 +8,5 @@
                 <geometry>
                     <mesh
-                        filename="package://morpheus_description/meshes/components/visual/HERAObstacleCourse.obj"
+                        filename="file://$(find morpheus_description)/meshes/components/visual/HERAObstacleCourse.obj"
                         scale="0.01 0.01 0.01" />
                 </geometry>
@@ -19,5 +19,5 @@
                 <geometry>
                     <mesh
-                        filename="package://morpheus_description/meshes/components/collision/HERAObstacleCourse.obj"
+                        filename="file://$(find morpheus_description)/meshes/components/collision/HERAObstacleCourse.obj"
                         scale="0.01 0.01 0.01" />
                 </geometry>

File: morpheus_description/urdf/macros/node2.xacro (robot description, xacro)
@@ -29,5 +29,5 @@
             <origin rpy="0 0 0" xyz="0 0 0"/>
             <geometry>
-                <mesh filename="package://morpheus_description/meshes/components/visual/PMA3.stl" scale="${scale * 0.001} ${scale * 0.001} ${scale * 0.001}"/>
+                <mesh filename="file://$(find morpheus_description)/meshes/components/visual/PMA3.stl" scale="${scale * 0.001} ${scale * 0.001} ${scale * 0.001}"/>
             </geometry>
             <material name="grey">
@@ -38,5 +38,5 @@
             <origin rpy="0 0 0" xyz="0 0 0" />
             <geometry>
-                <mesh filename="package://morpheus_description/meshes/components/collision/PMA3.stl" scale="${scale * 0.001} ${scale * 0.001} ${scale * 0.001}"/>
+                <mesh filename="file://$(find morpheus_description)/meshes/components/collision/PMA3.stl" scale="${scale * 0.001} ${scale * 0.001} ${scale * 0.001}"/>
             </geometry>
         </collision>

File: morpheus_description/urdf/macros/table_2x8ft.xacro (robot description, xacro)
@@ -12,5 +12,5 @@
             <origin rpy="-1.57079632679 0 0" xyz="0 0 ${-scale * 1}"/>
             <geometry>
-                <mesh filename="package://morpheus_description/meshes/components/visual/table_2x8ft.obj" scale="${scale} ${scale} ${scale}"/>
+                <mesh filename="file://$(find morpheus_description)/meshes/components/visual/table_2x8ft.obj" scale="${scale} ${scale} ${scale}"/>
             </geometry>
             <material name="grey">
@@ -21,5 +21,5 @@
             <origin rpy="-1.57079632679 0 0" xyz="0 0 ${-scale * 1}" />
             <geometry>
-                <mesh filename="package://morpheus_description/meshes/components/collision/table_2x8ft.obj" scale="${scale} ${scale} ${scale}"/>
+                <mesh filename="file://$(find morpheus_description)/meshes/components/collision/table_2x8ft.obj" scale="${scale} ${scale} ${scale}"/>
             </geometry>
         </collision>

File: morpheus_description/urdf/macros/teapot.xacro (robot description, xacro)
@@ -12,5 +12,5 @@
             <origin rpy="1.57079632679 0 0" xyz="0 0 0"/>
             <geometry>
-                <mesh filename="package://morpheus_description/meshes/components/visual/teapot.obj" scale="${scale} ${scale} ${scale}"/>
+                <mesh filename="file://$(find morpheus_description)/meshes/components/visual/teapot.obj" scale="${scale} ${scale} ${scale}"/>
             </geometry>
             <material name="grey">
@@ -21,5 +21,5 @@
             <origin rpy="1.57079632679 0 0" xyz="0 0 0" />
             <geometry>
-                <mesh filename="package://morpheus_description/meshes/components/collision/teapot.obj" scale="${scale} ${scale} ${scale}"/>
+                <mesh filename="file://$(find morpheus_description)/meshes/components/collision/teapot.obj" scale="${scale} ${scale} ${scale}"/>
             </geometry>
         </collision>

File: morpheus_description/urdf/macros/test_wall_1.xacro (robot description, xacro)
@@ -12,5 +12,5 @@
             <origin rpy="1.57079632679 0 0" xyz="0 0 0"/>
             <geometry>
-                <mesh filename="package://morpheus_description/meshes/components/visual/test_wall_1.obj" scale="${scale} ${scale} ${scale}"/>
+                <mesh filename="file://$(find morpheus_description)/meshes/components/visual/test_wall_1.obj" scale="${scale} ${scale} ${scale}"/>
             </geometry>
             <material name="grey">
@@ -21,5 +21,5 @@
             <origin rpy="1.57079632679 0 0" xyz="0 0 0" />
             <geometry>
-                <mesh filename="package://morpheus_description/meshes/components/collision/test_wall_1.obj" scale="${scale} ${scale} ${scale}"/>
+                <mesh filename="file://$(find morpheus_description)/meshes/components/collision/test_wall_1.obj" scale="${scale} ${scale} ${scale}"/>
             </geometry>
         </collision>

File: morpheus_description/urdf/macros/ur5e.xacro (robot description, xacro)
@@ -1,4 +1,4 @@
 <?xml version="1.0"?>
-<robot xmlns:xacro="http://wiki.ros.org/xacro" name="${name}">
+<robot xmlns:xacro="http://wiki.ros.org/xacro">
   <xacro:macro name="ur5e" params="
     *origin
@@ -41,22 +41,60 @@
     rw_rate:=0
     ">
+    <!-- Set up xacro args from macro params -->
+    <xacro:arg name="name" default="${name}" />
+    <xacro:arg name="ur_type" default="${ur_type}" />
+    <xacro:arg name="tf_prefix" default="${tf_prefix}" />
+    <xacro:arg name="parent" default="${parent}" />
+    <xacro:arg name="joint_limits_parameters_file" default="${joint_limits_parameters_file}" />
+    <xacro:arg name="kinematics_parameters_file" default="${kinematics_parameters_file}" />
+    <xacro:arg name="physical_parameters_file" default="${physical_parameters_file}" />
+    <xacro:arg name="visual_parameters_file" default="${visual_parameters_file}" />
+    <xacro:arg name="safety_limits" default="${safety_limits}" />
+    <xacro:arg name="safety_pos_margin" default="${safety_pos_margin}" />
+    <xacro:arg name="safety_k_position" default="${safety_k_position}" />
+    <xacro:arg name="force_abs_paths" default="${force_abs_paths}" />
+    <xacro:arg name="control" default="${control}" />
+    <xacro:arg name="gazebo" default="${gazebo}" />
+    <xacro:arg name="end_effector" default="${end_effector}" />
+    <xacro:arg name="simulation_controllers" default="${simulation_controllers}" />
+    <xacro:arg name="ros_namespace" default="${ros_namespace}" />
+    <xacro:arg name="initial_positions_file" default="${initial_positions_file}" />
+    <xacro:arg name="robot_ip" default="${robot_ip}" />
+    <xacro:arg name="script_filename" default="${script_filename}" />
+    <xacro:arg name="input_recipe_filename" default="${input_recipe_filename}" />
+    <xacro:arg name="output_recipe_filename" default="${output_recipe_filename}" />
+    <xacro:arg name="transmission_hw_interface" default="${transmission_hw_interface}" />
+    <xacro:arg name="use_mock_hardware" default="${use_mock_hardware}" />
+    <xacro:arg name="mock_sensor_commands" default="${mock_sensor_commands}" />
+    <xacro:arg name="headless_mode" default="${headless_mode}" />
+    <xacro:arg name="initial_positions" default="${initial_positions}" />
+    <xacro:arg name="use_tool_communication" default="${use_tool_communication}" />
+    <xacro:arg name="tool_voltage" default="${tool_voltage}" />
+    <xacro:arg name="tool_parity" default="${tool_parity}" />
+    <xacro:arg name="tool_baud_rate" default="${tool_baud_rate}" />
+    <xacro:arg name="tool_stop_bits" default="${tool_stop_bits}" />
+    <xacro:arg name="tool_rx_idle_chars" default="${tool_rx_idle_chars}" />
+    <xacro:arg name="tool_tx_idle_chars" default="${tool_tx_idle_chars}" />
+    <xacro:arg name="tool_device_name" default="${tool_device_name}" />
+    <xacro:arg name="tool_tcp_port" default="${tool_tcp_port}" />
+    <xacro:arg name="reverse_port" default="${reverse_port}" />
+    <xacro:arg name="script_sender_port" default="${script_sender_port}" />
+    <xacro:arg name="reverse_ip" default="${reverse_ip}" />
+    <xacro:arg name="script_command_port" default="${script_command_port}" />
+    <xacro:arg name="trajectory_port" default="${trajectory_port}" />
+    <xacro:arg name="non_blocking_read" default="${non_blocking_read}" />
+    <xacro:arg name="robot_receive_timeout" default="${robot_receive_timeout}" />
+    <xacro:arg name="rw_rate" default="${rw_rate}" />
     <xacro:if value="${control}">
       <xacro:if value="${gazebo}">
-        <xacro:include filename="$(find ur_simulation_gz)/urdf/ur_gz.urdf.xacro" />
+        <xacro:include filename="$(find ur_simulation_gz)/urdf/ur_gz.urdf.xacro" ns="include"/>
       </xacro:if>
       <xacro:unless value="${gazebo}">
-        <xacro:include filename="$(find ur_robot_driver)/urdf/ur.urdf.xacro" />
+        <xacro:include filename="$(find ur_robot_driver)/urdf/ur.urdf.xacro" ns="include"/>
       </xacro:unless>
     </xacro:if>
     <xacro:unless value="${control}">
-      <xacro:include filename="$(find ur_description)/urdf/ur.urdf.xacro" />
+      <xacro:include filename="$(find ur_description)/urdf/ur.urdf.xacro" ns="include"/>
     </xacro:unless>
-    <!-- Add an additional link to plan with. Oriented like the Trossen ee_gripper_link frame. -->
-    <link name="${tf_prefix}tcp_link" />
-    <joint name="${tf_prefix}tcp_joint" type="fixed">
-      <parent link="${tf_prefix}wrist_3_link" />
-      <child link="${tf_prefix}tcp_link" />
-      <origin rpy="0 ${-pi/2} ${-pi/2}" xyz="0 0 ${tcp_offset}" />
-    </joint>
   </xacro:macro>
 </robot>

File: morpheus_description/urdf/macros/ur5e_macro.xacro (robot description, xacro)
@@ -7,5 +7,4 @@
     tf_prefix
     parent
-    joint_limits_parameters_file:='$(find ur_description)/config/ur5e/joint_limits.yaml'
     tcp_offset
     *origin">
@@ -16,5 +15,5 @@
       tf_prefix="${tf_prefix}"
       parent="${parent}"
-      joint_limits_parameters_file="${joint_limits_parameters_file}"
+      joint_limits_parameters_file="$(find ur_description)/config/ur5e/joint_limits.yaml"
       kinematics_parameters_file='$(find ur_description)/config/ur5e/default_kinematics.yaml'
       physical_parameters_file='$(find ur_description)/config/ur5e/physical_parameters.yaml'
@@ -23,4 +22,5 @@
       safety_pos_margin="0.15"
       safety_k_position="20"
+      force_abs_paths="true"
       >
       <xacro:insert_block name="origin" />

File: morpheus_description/urdf/macros/wall.xacro (robot description, xacro)
@@ -12,5 +12,5 @@
             <origin rpy="1.57079632679 0 0" xyz="0 0 0"/>
             <geometry>
-                <mesh filename="package://morpheus_description/meshes/components/visual/wall.obj" scale="${scale} ${scale} ${scale}"/>
+                <mesh filename="file://$(find morpheus_description)/meshes/components/visual/wall.obj" scale="${scale} ${scale} ${scale}"/>
             </geometry>
             <material name="grey">
@@ -21,5 +21,5 @@
             <origin rpy="1.57079632679 0 0" xyz="0 0 0" />
             <geometry>
-                <mesh filename="package://morpheus_description/meshes/components/collision/wall.obj" scale="${scale} ${scale} ${scale}"/>
+                <mesh filename="file://$(find morpheus_description)/meshes/components/collision/wall.obj" scale="${scale} ${scale} ${scale}"/>
             </geometry>
         </collision>

File: morpheus_description/urdf/macros/wall_4x12in.xacro (robot description, xacro)
@@ -12,5 +12,5 @@
             <origin rpy="0 0 1.57079632679" xyz="${scale * 12} 0.0 0.0"/>
             <geometry>
-                <mesh filename="package://morpheus_description/meshes/components/visual/wall_4x12in.obj" scale="${scale} ${scale} ${scale}"/>
+                <mesh filename="file://$(find morpheus_description)/meshes/components/visual/wall_4x12in.obj" scale="${scale} ${scale} ${scale}"/>
             </geometry>
             <material name="grey">
@@ -21,5 +21,5 @@
             <origin rpy="0 0 1.57079632679" xyz="${scale * 12} 0.0 0.0"/>
             <geometry>
-                <mesh filename="package://morpheus_description/meshes/components/collision/wall_4x12in.obj" scale="${scale} ${scale} ${scale}"/>
+                <mesh filename="file://$(find morpheus_description)/meshes/components/collision/wall_4x12in.obj" scale="${scale} ${scale} ${scale}"/>
             </geometry>
         </collision>

File: morpheus_description/urdf/macros/wall_6x12in.xacro (robot description, xacro)
@@ -12,5 +12,5 @@
             <origin rpy="0 0 1.57079632679" xyz="${scale * 12} 0.0 0.0"/>
             <geometry>
-                <mesh filename="package://morpheus_description/meshes/components/visual/wall_6x12in.obj" scale="${scale} ${scale} ${scale}"/>
+                <mesh filename="file://$(find morpheus_description)/meshes/components/visual/wall_6x12in.obj" scale="${scale} ${scale} ${scale}"/>
             </geometry>
             <material name="grey">
@@ -21,5 +21,5 @@
             <origin rpy="0 0 1.57079632679" xyz="${scale * 12} 0.0 0.0"/>
             <geometry>
-                <mesh filename="package://morpheus_description/meshes/components/collision/wall_6x12in.obj" scale="${scale} ${scale} ${scale}"/>
+                <mesh filename="file://$(find morpheus_description)/meshes/components/collision/wall_6x12in.obj" scale="${scale} ${scale} ${scale}"/>
             </geometry>
         </collision>

File: morpheus_description/urdf/scenes/a_bot_scene.xacro (robot description, xacro)
@@ -1,7 +1,4 @@
 <?xml version="1.0"?>
-<robot xmlns:xacro="http://www.ros.org/wiki/xacro" name="a_bot_scene">
-    <xacro:arg name="joint_limits_parameters_file"
-        default="$(find ur_description)/config/ur5e/joint_limits.yaml" />
-    <xacro:arg name="transmission_hw_interface" default="hardware_interface/PositionJointInterface" />
+<robot xmlns:xacro="http://www.ros.org/wiki/xacro" name="ur">
     <link name="world" />
     <xacro:include filename="$(find morpheus_description)/urdf/macros/simple_pedestal_macro.xacro" />
@@ -16,6 +13,4 @@
         prefix=""
         parent="world"
-        transmission_hw_interface="$(arg transmission_hw_interface)"
-        joint_limits_parameters_file="$(arg joint_limits_parameters_file)"
     >
         <origin xyz="0 0 ${0.0254 * 34.75}" rpy="0 0 0" />
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