Commit message: ROS2 Migration: UR robot URDF/SRDF rework WIP, low latency Linux kernel install added, considering realtime kernel install as part of Dockerfile

File: morpheus_description/urdf/macros/Test_Block_1.xacro (robot description, xacro)
@@ -12,5 +12,5 @@
             <origin rpy="0 0 0" xyz="0 0 0"/>
             <geometry>
-                <mesh filename="file://$(find morpheus_description)/meshes/components/visual/test_block_1.stl" scale="${scale} ${scale} ${scale}"/>
+                <mesh filename="file://$(find morpheus_description)/meshes/visual/test_block_1.stl" scale="${scale} ${scale} ${scale}"/>
             </geometry>
             <material name="grey">
@@ -21,5 +21,5 @@
             <origin rpy="0 0 0" xyz="0 0 0" />
             <geometry>
-                <mesh filename="file://$(find morpheus_description)/meshes/components/collision/test_block_1.stl" scale="${scale} ${scale} ${scale}"/>
+                <mesh filename="file://$(find morpheus_description)/meshes/collision/test_block_1.stl" scale="${scale} ${scale} ${scale}"/>
             </geometry>
         </collision>

File: morpheus_description/urdf/macros/a_bot_macro.xacro (robot description, xacro)
@@ -3,10 +3,12 @@
     <xacro:include filename="$(find morpheus_description)/urdf/macros/ur5e_macro.xacro" />
     <xacro:include filename="$(find morpheus_description)/urdf/macros/d415_mount_macro.xacro" />
-    <xacro:include filename="$(find robotiq_2f_85_gripper_description)/urdf/robotiq_arg2f_85_macro.xacro" />
+    <xacro:include filename="$(find robotiq_description)/urdf/robotiq_2f_85_macro.urdf.xacro" />
     <xacro:macro name="a_bot"
         params="
         prefix
         parent
-        *origin">
+        *origin
+        use_fake_hardware:=false
+        ">
         <xacro:ur5e
             tf_prefix="${prefix}"
@@ -22,12 +24,12 @@
             <origin xyz="0 0 0" rpy="0 0 0" />
         </xacro:d415_mount>
-        <xacro:robotiq_arg2f_85
+        <xacro:robotiq_gripper
+            name="${prefix}robotiq_2f_85"
             prefix="${prefix}"
             parent="${prefix}d415_mount_attach_link"
-            transmission_hw_interface="hardware_interface/PositionJointInterface"
-            add_cable_protector="true"
+            use_fake_hardware="${use_fake_hardware}"
         >
             <origin xyz="0 0 0.003" rpy="0 0 ${pi}" />
-        </xacro:robotiq_arg2f_85>
+        </xacro:robotiq_gripper>
     </xacro:macro>
 </robot>

File: morpheus_description/urdf/macros/b_bot_macro.xacro (robot description, xacro)
@@ -3,10 +3,12 @@
     <xacro:include filename="$(find morpheus_description)/urdf/macros/ur5e_macro.xacro" />
     <xacro:include filename="$(find morpheus_description)/urdf/macros/d415_mount_macro.xacro" />
-    <xacro:include filename="$(find onrobot_rg2ft_description)/urdf/onrobot_rg2ft_macro.xacro" />
+    <xacro:include filename="$(find onrobot_description)/urdf/onrobot_macro.xacro" />
     <xacro:macro name="b_bot"
         params="
         prefix
         parent
-        *origin">
+        *origin
+        use_fake_hardware:=false
+        ">
         <xacro:ur5e
             tf_prefix="${prefix}"
@@ -22,11 +24,17 @@
             <origin xyz="0 0 0" rpy="0 0 0" />
         </xacro:d415_mount>
-        <xacro:onrobot_rg2ft
+        <xacro:onrobot
+            onrobot_type="rg2"
             prefix="${prefix}"
-            parent="${prefix}d415_mount_attach_link"
-            hw_interface="hardware_interface/PositionJointInterface"
+            use_fake_hardware="${use_fake_hardware}"
         >
             <origin xyz="0 0 0.0026" rpy="0 0 ${pi}" />
-        </xacro:onrobot_rg2ft>
+        </xacro:onrobot>
+        <!-- Connect the OnRobot to the UR robot -->
+        <joint name="${prefix}onrobot_base_link_joint" type="fixed">
+            <parent link="${prefix}tool0"/>
+            <child link="${prefix}onrobot_base_link"/>
+            <origin xyz="0 0 0" rpy="0 0 ${-pi/2}"/>
+        </joint>
     </xacro:macro>
 </robot>

File: morpheus_description/urdf/macros/bar_12in.xacro (robot description, xacro)
@@ -12,5 +12,5 @@
             <origin rpy="0 0 0" xyz="0 0 0"/>
             <geometry>
-                <mesh filename="file://$(find morpheus_description)/meshes/components/visual/bar_12in.obj" scale="${scale} ${scale} ${scale}"/>
+                <mesh filename="file://$(find morpheus_description)/meshes/visual/bar_12in.obj" scale="${scale} ${scale} ${scale}"/>
             </geometry>
             <material name="grey">
@@ -21,5 +21,5 @@
             <origin rpy="0 0 0" xyz="0 0 0" />
             <geometry>
-                <mesh filename="file://$(find morpheus_description)/meshes/components/collision/bar_12in.obj" scale="${scale} ${scale} ${scale}"/>
+                <mesh filename="file://$(find morpheus_description)/meshes/collision/bar_12in.obj" scale="${scale} ${scale} ${scale}"/>
             </geometry>
         </collision>

File: morpheus_description/urdf/macros/bar_4in.xacro (robot description, xacro)
@@ -12,5 +12,5 @@
             <origin rpy="1.57079632679 0 0" xyz="0 ${scale * 1} 0"/>
             <geometry>
-                <mesh filename="file://$(find morpheus_description)/meshes/components/visual/bar_4in.obj" scale="${scale} ${scale} ${scale}"/>
+                <mesh filename="file://$(find morpheus_description)/meshes/visual/bar_4in.obj" scale="${scale} ${scale} ${scale}"/>
             </geometry>
             <material name="grey">
@@ -21,5 +21,5 @@
             <origin rpy="1.57079632679 0 0" xyz="0 ${scale * 1} 0" />
             <geometry>
-                <mesh filename="file://$(find morpheus_description)/meshes/components/collision/bar_4in.obj" scale="${scale} ${scale} ${scale}"/>
+                <mesh filename="file://$(find morpheus_description)/meshes/collision/bar_4in.obj" scale="${scale} ${scale} ${scale}"/>
             </geometry>
         </collision>

File: morpheus_description/urdf/macros/block.xacro (robot description, xacro)
@@ -12,5 +12,5 @@
             <origin rpy="1.57079632679 0 0" xyz="0 0 0"/>
             <geometry>
-                <mesh filename="file://$(find morpheus_description)/meshes/components/visual/block.obj" scale="${scale} ${scale} ${scale}"/>
+                <mesh filename="file://$(find morpheus_description)/meshes/visual/block.obj" scale="${scale} ${scale} ${scale}"/>
             </geometry>
             <material name="grey">
@@ -21,5 +21,5 @@
             <origin rpy="1.57079632679 0 0" xyz="0 0 0" />
             <geometry>
-                <mesh filename="file://$(find morpheus_description)/meshes/components/collision/block.obj" scale="${scale} ${scale} ${scale}"/>
+                <mesh filename="file://$(find morpheus_description)/meshes/collision/block.obj" scale="${scale} ${scale} ${scale}"/>
             </geometry>
         </collision>

File: morpheus_description/urdf/macros/dragon_simple.xacro (robot description, xacro)
@@ -12,5 +12,5 @@
             <origin rpy="1.57079632679 0 0" xyz="0 0 0"/>
             <geometry>
-                <mesh filename="file://$(find morpheus_description)/meshes/components/visual/dragon_simple.obj" scale="${scale} ${scale} ${scale}"/>
+                <mesh filename="file://$(find morpheus_description)/meshes/visual/dragon_simple.obj" scale="${scale} ${scale} ${scale}"/>
             </geometry>
             <material name="grey">
@@ -21,5 +21,5 @@
             <origin rpy="1.57079632679 0 0" xyz="0 0 0" />
             <geometry>
-                <mesh filename="file://$(find morpheus_description)/meshes/components/collision/dragon_simple.obj" scale="${scale} ${scale} ${scale}"/>
+                <mesh filename="file://$(find morpheus_description)/meshes/collision/dragon_simple.obj" scale="${scale} ${scale} ${scale}"/>
             </geometry>
         </collision>

File: morpheus_description/urdf/macros/foam.xacro (robot description, xacro)
@@ -12,5 +12,5 @@
             <origin rpy="1.57079632679 0 0" xyz="0 0 0"/>
             <geometry>
-                <mesh filename="file://$(find morpheus_description)/meshes/components/visual/foam.obj" scale="${scale} ${scale} ${scale}"/>
+                <mesh filename="file://$(find morpheus_description)/meshes/visual/foam.obj" scale="${scale} ${scale} ${scale}"/>
             </geometry>
             <material name="grey">
@@ -21,5 +21,5 @@
             <origin rpy="1.57079632679 0 0" xyz="0 0 0" />
             <geometry>
-                <mesh filename="file://$(find morpheus_description)/meshes/components/collision/foam.obj" scale="${scale} ${scale} ${scale}"/>
+                <mesh filename="file://$(find morpheus_description)/meshes/collision/foam.obj" scale="${scale} ${scale} ${scale}"/>
             </geometry>
         </collision>

File: morpheus_description/urdf/macros/hera_obstacle_course_mesh.xacro (robot description, xacro)
@@ -8,5 +8,5 @@
                 <geometry>
                     <mesh
-                        filename="file://$(find morpheus_description)/meshes/components/visual/HERAObstacleCourse.obj"
+                        filename="file://$(find morpheus_description)/meshes/visual/HERAObstacleCourse.obj"
                         scale="0.01 0.01 0.01" />
                 </geometry>
@@ -19,5 +19,5 @@
                 <geometry>
                     <mesh
-                        filename="file://$(find morpheus_description)/meshes/components/collision/HERAObstacleCourse.obj"
+                        filename="file://$(find morpheus_description)/meshes/collision/HERAObstacleCourse.obj"
                         scale="0.01 0.01 0.01" />
                 </geometry>

File: morpheus_description/urdf/macros/node2.xacro (robot description, xacro)
@@ -29,5 +29,5 @@
             <origin rpy="0 0 0" xyz="0 0 0"/>
             <geometry>
-                <mesh filename="file://$(find morpheus_description)/meshes/components/visual/PMA3.stl" scale="${scale * 0.001} ${scale * 0.001} ${scale * 0.001}"/>
+                <mesh filename="file://$(find morpheus_description)/meshes/visual/PMA3.stl" scale="${scale * 0.001} ${scale * 0.001} ${scale * 0.001}"/>
             </geometry>
             <material name="grey">
@@ -38,5 +38,5 @@
             <origin rpy="0 0 0" xyz="0 0 0" />
             <geometry>
-                <mesh filename="file://$(find morpheus_description)/meshes/components/collision/PMA3.stl" scale="${scale * 0.001} ${scale * 0.001} ${scale * 0.001}"/>
+                <mesh filename="file://$(find morpheus_description)/meshes/collision/PMA3.stl" scale="${scale * 0.001} ${scale * 0.001} ${scale * 0.001}"/>
             </geometry>
         </collision>

File: morpheus_description/urdf/macros/table_2x8ft.xacro (robot description, xacro)
@@ -12,5 +12,5 @@
             <origin rpy="-1.57079632679 0 0" xyz="0 0 ${-scale * 1}"/>
             <geometry>
-                <mesh filename="file://$(find morpheus_description)/meshes/components/visual/table_2x8ft.obj" scale="${scale} ${scale} ${scale}"/>
+                <mesh filename="file://$(find morpheus_description)/meshes/visual/table_2x8ft.obj" scale="${scale} ${scale} ${scale}"/>
             </geometry>
             <material name="grey">
@@ -21,5 +21,5 @@
             <origin rpy="-1.57079632679 0 0" xyz="0 0 ${-scale * 1}" />
             <geometry>
-                <mesh filename="file://$(find morpheus_description)/meshes/components/collision/table_2x8ft.obj" scale="${scale} ${scale} ${scale}"/>
+                <mesh filename="file://$(find morpheus_description)/meshes/collision/table_2x8ft.obj" scale="${scale} ${scale} ${scale}"/>
             </geometry>
         </collision>

File: morpheus_description/urdf/macros/teapot.xacro (robot description, xacro)
@@ -12,5 +12,5 @@
             <origin rpy="1.57079632679 0 0" xyz="0 0 0"/>
             <geometry>
-                <mesh filename="file://$(find morpheus_description)/meshes/components/visual/teapot.obj" scale="${scale} ${scale} ${scale}"/>
+                <mesh filename="file://$(find morpheus_description)/meshes/visual/teapot.obj" scale="${scale} ${scale} ${scale}"/>
             </geometry>
             <material name="grey">
@@ -21,5 +21,5 @@
             <origin rpy="1.57079632679 0 0" xyz="0 0 0" />
             <geometry>
-                <mesh filename="file://$(find morpheus_description)/meshes/components/collision/teapot.obj" scale="${scale} ${scale} ${scale}"/>
+                <mesh filename="file://$(find morpheus_description)/meshes/collision/teapot.obj" scale="${scale} ${scale} ${scale}"/>
             </geometry>
         </collision>

File: morpheus_description/urdf/macros/test_wall_1.xacro (robot description, xacro)
@@ -12,5 +12,5 @@
             <origin rpy="1.57079632679 0 0" xyz="0 0 0"/>
             <geometry>
-                <mesh filename="file://$(find morpheus_description)/meshes/components/visual/test_wall_1.obj" scale="${scale} ${scale} ${scale}"/>
+                <mesh filename="file://$(find morpheus_description)/meshes/visual/test_wall_1.obj" scale="${scale} ${scale} ${scale}"/>
             </geometry>
             <material name="grey">
@@ -21,5 +21,5 @@
             <origin rpy="1.57079632679 0 0" xyz="0 0 0" />
             <geometry>
-                <mesh filename="file://$(find morpheus_description)/meshes/components/collision/test_wall_1.obj" scale="${scale} ${scale} ${scale}"/>
+                <mesh filename="file://$(find morpheus_description)/meshes/collision/test_wall_1.obj" scale="${scale} ${scale} ${scale}"/>
             </geometry>
         </collision>

File: morpheus_description/urdf/macros/ur5e_macro.xacro (robot description, xacro)
@@ -2,35 +2,35 @@
 <!-- This macro adds a convenient TF frame at the tip of the closed gripper. -->
 <!-- The position of the TF frame has not been measured at all and needs to be calibrated. -->
-<robot name="ur5e" xmlns:xacro="http://www.ros.org/wiki/xacro">
-  <xacro:macro name="ur5e" params="
-    name:='ur5e'
-    tf_prefix
-    parent
-    tcp_offset
-    *origin">
-    <!-- ur5e -->
+<robot xmlns:xacro="http://www.ros.org/wiki/xacro">
     <xacro:include filename="$(find ur_description)/urdf/ur_macro.xacro" />
-    <xacro:ur_robot
-      name="${name}"
-      tf_prefix="${tf_prefix}"
-      parent="${parent}"
-      joint_limits_parameters_file="$(find ur_description)/config/ur5e/joint_limits.yaml"
-      kinematics_parameters_file='$(find ur_description)/config/ur5e/default_kinematics.yaml'
-      physical_parameters_file='$(find ur_description)/config/ur5e/physical_parameters.yaml'
-      visual_parameters_file='$(find ur_description)/config/ur5e/visual_parameters.yaml'
-      safety_limits="false"
-      safety_pos_margin="0.15"
-      safety_k_position="20"
-      force_abs_paths="true"
-      >
-      <xacro:insert_block name="origin" />
-    </xacro:ur_robot>
-    <!-- Add an additional link to plan with. Oriented like the Trossen ee_gripper_link frame. -->
-    <link name="${tf_prefix}tcp_link" />
-    <joint name="${tf_prefix}tcp_joint" type="fixed">
-      <parent link="${tf_prefix}wrist_3_link" />
-      <child link="${tf_prefix}tcp_link" />
-      <origin rpy="0 ${-pi/2} ${-pi/2}" xyz="0 0 ${tcp_offset}" />
-    </joint>
-  </xacro:macro>
+    <xacro:macro name="ur5e" params="
+        name:='ur5e'
+        tf_prefix
+        parent
+        tcp_offset
+        *origin">
+        <!-- ur5e -->
+        <xacro:ur_robot
+            name="${name}"
+            tf_prefix="${tf_prefix}"
+            parent="${parent}"
+            joint_limits_parameters_file="$(find ur_description)/config/ur5e/joint_limits.yaml"
+            kinematics_parameters_file='$(find ur_description)/config/ur5e/default_kinematics.yaml'
+            physical_parameters_file='$(find ur_description)/config/ur5e/physical_parameters.yaml'
+            visual_parameters_file='$(find ur_description)/config/ur5e/visual_parameters.yaml'
+            safety_limits="false"
+            safety_pos_margin="0.15"
+            safety_k_position="20"
+            force_abs_paths="true"
+            >
+            <xacro:insert_block name="origin" />
+        </xacro:ur_robot>
+        <!-- Add an additional link to plan with. Oriented like the Trossen ee_gripper_link frame. -->
+        <link name="${tf_prefix}tcp_link" />
+        <joint name="${tf_prefix}tcp_joint" type="fixed">
+            <parent link="${tf_prefix}wrist_3_link" />
+            <child link="${tf_prefix}tcp_link" />
+            <origin rpy="0 ${-pi/2} ${-pi/2}" xyz="0 0 ${tcp_offset}" />
+        </joint>
+    </xacro:macro>
 </robot>

File: morpheus_description/urdf/macros/wall.xacro (robot description, xacro)
@@ -12,5 +12,5 @@
             <origin rpy="1.57079632679 0 0" xyz="0 0 0"/>
             <geometry>
-                <mesh filename="file://$(find morpheus_description)/meshes/components/visual/wall.obj" scale="${scale} ${scale} ${scale}"/>
+                <mesh filename="file://$(find morpheus_description)/meshes/visual/wall.obj" scale="${scale} ${scale} ${scale}"/>
             </geometry>
             <material name="grey">
@@ -21,5 +21,5 @@
             <origin rpy="1.57079632679 0 0" xyz="0 0 0" />
             <geometry>
-                <mesh filename="file://$(find morpheus_description)/meshes/components/collision/wall.obj" scale="${scale} ${scale} ${scale}"/>
+                <mesh filename="file://$(find morpheus_description)/meshes/collision/wall.obj" scale="${scale} ${scale} ${scale}"/>
             </geometry>
         </collision>

File: morpheus_description/urdf/macros/wall_4x12in.xacro (robot description, xacro)
@@ -12,5 +12,5 @@
             <origin rpy="0 0 1.57079632679" xyz="${scale * 12} 0.0 0.0"/>
             <geometry>
-                <mesh filename="file://$(find morpheus_description)/meshes/components/visual/wall_4x12in.obj" scale="${scale} ${scale} ${scale}"/>
+                <mesh filename="file://$(find morpheus_description)/meshes/visual/wall_4x12in.obj" scale="${scale} ${scale} ${scale}"/>
             </geometry>
             <material name="grey">
@@ -21,5 +21,5 @@
             <origin rpy="0 0 1.57079632679" xyz="${scale * 12} 0.0 0.0"/>
             <geometry>
-                <mesh filename="file://$(find morpheus_description)/meshes/components/collision/wall_4x12in.obj" scale="${scale} ${scale} ${scale}"/>
+                <mesh filename="file://$(find morpheus_description)/meshes/collision/wall_4x12in.obj" scale="${scale} ${scale} ${scale}"/>
             </geometry>
         </collision>

File: morpheus_description/urdf/macros/wall_6x12in.xacro (robot description, xacro)
@@ -12,5 +12,5 @@
             <origin rpy="0 0 1.57079632679" xyz="${scale * 12} 0.0 0.0"/>
             <geometry>
-                <mesh filename="file://$(find morpheus_description)/meshes/components/visual/wall_6x12in.obj" scale="${scale} ${scale} ${scale}"/>
+                <mesh filename="file://$(find morpheus_description)/meshes/visual/wall_6x12in.obj" scale="${scale} ${scale} ${scale}"/>
             </geometry>
             <material name="grey">
@@ -21,5 +21,5 @@
             <origin rpy="0 0 1.57079632679" xyz="${scale * 12} 0.0 0.0"/>
             <geometry>
-                <mesh filename="file://$(find morpheus_description)/meshes/components/collision/wall_6x12in.obj" scale="${scale} ${scale} ${scale}"/>
+                <mesh filename="file://$(find morpheus_description)/meshes/collision/wall_6x12in.obj" scale="${scale} ${scale} ${scale}"/>
             </geometry>
         </collision>

File: morpheus_description/urdf/scenes/a_bot_scene.xacro (robot description, xacro)
@@ -1,4 +1,5 @@
 <?xml version="1.0"?>
 <robot xmlns:xacro="http://www.ros.org/wiki/xacro" name="ur">
+    <xacro:arg name="use_fake_hardware" default = "true"/>
     <link name="world" />
     <xacro:include filename="$(find morpheus_description)/urdf/macros/simple_pedestal_macro.xacro" />
@@ -13,4 +14,5 @@
         prefix=""
         parent="world"
+        use_fake_hardware="$(arg use_fake_hardware)"
     >
         <origin xyz="0 0 ${0.0254 * 34.75}" rpy="0 0 0" />

File: morpheus_description/urdf/scenes/b_bot_scene.xacro (robot description, xacro)
@@ -1,4 +1,5 @@
 <?xml version="1.0"?>
 <robot xmlns:xacro="http://www.ros.org/wiki/xacro" name="ur">
+    <xacro:arg name="use_fake_hardware" default = "true"/>
     <link name="world" />
     <xacro:include filename="$(find morpheus_description)/urdf/macros/simple_pedestal_macro.xacro" />
@@ -13,4 +14,5 @@
         prefix=""
         parent="world"
+        use_fake_hardware="$(arg use_fake_hardware)"
     >
         <origin xyz="0 0 ${0.0254 * 34.75}" rpy="0 0 0" />

File: morpheus_sim/urdf/ur_gz.urdf.xacro (robot description, xacro)
@@ -6,5 +6,5 @@
   <xacro:include filename="$(find ur_simulation_gz)/urdf/ur_gz.ros2_control.xacro" />
   <!-- Arguments -->
-  <xacro:arg name="tf_prefix" default="" />
+  <xacro:arg name="tf_prefix" default=""/>
   <xacro:arg name="joint_limit_params" default="$(find ur_description)/config/$(arg ur_type)/joint_limits.yaml"/>
   <xacro:arg name="kinematics_params" default="$(find ur_description)/config/$(arg ur_type)/default_kinematics.yaml"/>
@@ -15,7 +15,7 @@
   <xacro:arg name="safety_pos_margin" default="0.15"/>
   <xacro:arg name="safety_k_position" default="20"/>
-  <xacro:arg name="simulation_controllers" default="" />
-  <xacro:arg name="ros_namespace" default="" />
-  <xacro:arg name="description_file" default="$(find morpheus_description)/urdf/scenes/b_bot_scene.xacro" />
+  <xacro:arg name="simulation_controllers" default=""/>
+  <xacro:arg name="ros_namespace" default=""/>
+  <xacro:arg name="description_file" default="$(find morpheus_description)/urdf/scenes/a_bot_scene.xacro"/>
   <!-- Create the scene containing the UR robot -->
   <xacro:include filename="$(arg description_file)"/>
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