Commit message: URDF tweaks to make a computationally cheaper version of dragon capsule for collision detection

File: morpheus_description/urdf/macros/dragon_simple.xacro (robot description, xacro)
@@ -2,8 +2,9 @@
 <robot name="dragon_simple" xmlns:xacro="http://www.ros.org/wiki/xacro">
   <xacro:macro name="dragon_simple"
-    params="x:=0 y:=0 z:=0 R:=0 P:=0 Y:=0 scale:=0.0254 prefix parent">
+    params="x:=0 y:=0 z:=0 R:=0 P:=0 Y:=0 scale:=1 prefix parent">
+    <xacro:property name="scale_mm" value="${scale * 0.0254}"/>
     <link name="${prefix}dragon_simple">
         <inertial>
-            <origin rpy="0 0 0" xyz="${scale * 0.0} ${scale * 0.0} ${scale * 2}"/>
+            <origin rpy="0 0 0" xyz="${scale_mm * 0.0} ${scale_mm * 0.0} ${scale_mm * 2}"/>
             <mass value="0.05"/>
             <inertia ixx="5" ixy="0" ixz="0" iyy="5" iyz="0" izz="12"/>
@@ -12,5 +13,5 @@
             <origin rpy="1.57079632679 0 0" xyz="0 0 0"/>
             <geometry>
-                <mesh filename="file://$(find morpheus_description)/meshes/visual/dragon_simple.obj" scale="${scale} ${scale} ${scale}"/>
+                <mesh filename="file://$(find morpheus_description)/meshes/visual/dragon_simple.obj" scale="${scale_mm} ${scale_mm} ${scale_mm}"/>
             </geometry>
             <material name="grey">
@@ -21,5 +22,5 @@
             <origin rpy="1.57079632679 0 0" xyz="0 0 0" />
             <geometry>
-                <mesh filename="file://$(find morpheus_description)/meshes/collision/dragon_simple.obj" scale="${scale} ${scale} ${scale}"/>
+                <mesh filename="file://$(find morpheus_description)/meshes/collision/dragon_simple.obj" scale="${scale_mm} ${scale_mm} ${scale_mm}"/>
             </geometry>
         </collision>

File: morpheus_driver/urdf/ur_endeffector_control.urdf.xacro (robot description, xacro)
@@ -67,5 +67,5 @@
     <xacro:arg name="port" default="502"/>
     <!-- Additional URDF Files -->
-    <xacro:arg name="environment_file" default="$(find morpheus_description)/urdf/scenes/node2_scene.xacro" />
+    <xacro:arg name="environment_file" default="$(find morpheus_description)/urdf/scenes/node2_dragon_scene.xacro" />
     <!-- Robot Include -->
     <xacro:include filename="$(find morpheus_description)/urdf/macros/ur_endeffector_macro.xacro" />
