Commit message: URDF tweaks for consistency and readability. Modification of URDF scene with Node2 and Dragon to clearly show distance field markers/vectors.

File: morpheus_description/urdf/macros/hab_table.xacro (robot description, xacro)
@@ -2,5 +2,12 @@
 <robot name="hab_table" xmlns:xacro="http://ros.org/wiki/xacro">
   <xacro:macro name="hab_table"
-      params="x:=0 y:=0 z:=0 R:=0 P:=0 Y:=0 length:=${91 * 0.0254} width:=${48 * 0.0254} height:=0.0254 scale:=1 prefix parent">
+    params="
+    length:=${91 * 0.0254}
+    width:=${48 * 0.0254}
+    height:=${1 * 0.0254}
+    scale:=1
+    prefix
+    parent
+    *origin">
     <link name="${prefix}hab_table">
       <visual>
@@ -23,5 +30,5 @@
         <parent link="${parent}" />
         <child link="${prefix}hab_table" />
-        <origin xyz="${x} ${y} ${z}" rpy="${R} ${P} ${Y}" />
+        <xacro:insert_block name="origin" />
     </joint>
   </xacro:macro>

File: morpheus_description/urdf/macros/hera_table.xacro (robot description, xacro)
@@ -2,5 +2,12 @@
 <robot name="hera_table" xmlns:xacro="http://ros.org/wiki/xacro">
   <xacro:macro name="hera_table"
-      params="x:=0 y:=0 z:=0 R:=0 P:=0 Y:=0 length:=${36 * 0.0254} width:=${24 * 0.0254} height:=0.0254 scale:=1 prefix parent">
+    params="
+    length:=${36 * 0.0254}
+    width:=${24 * 0.0254}
+    height:=${1 * 0.0254}
+    scale:=1
+    prefix
+    parent
+    *origin">
     <link name="${prefix}hera_table">
       <visual>
@@ -23,5 +30,5 @@
         <parent link="${parent}" />
         <child link="${prefix}hera_table" />
-        <origin xyz="${x} ${y} ${z}" rpy="${R} ${P} ${Y}" />
+        <xacro:insert_block name="origin" />
     </joint>
   </xacro:macro>

File: morpheus_description/urdf/macros/node2.xacro (robot description, xacro)
@@ -2,8 +2,14 @@
 <robot name="node2" xmlns:xacro="http://ros.org/wiki/xacro">
   <xacro:macro name="node2"
-      params="x:=0 y:=0 z:=0 R:=0 P:=0 Y:=0 height:=0.3683 radius:=0.1080 scale:=1 prefix parent">
+    params="
+    prefix
+    parent
+    height:=0.335
+    radius:=0.11
+    scale:=1
+    *origin">
     <link name="${prefix}node2">
       <visual>
-        <origin xyz="${-height / 2} 0 0" rpy="0 ${pi / 2} 0"/>
+        <origin xyz="0 ${height / 2} 0" rpy="${pi / 2} 0 0"/>
         <geometry>
           <cylinder length="${height * scale}" radius="${radius * scale}"/>
@@ -14,5 +20,5 @@
       </visual>
       <collision>
-        <origin xyz="${-height / 2} 0 0" rpy="0 ${pi / 2} 0"/>
+        <origin xyz="0 ${height / 2} 0" rpy="${pi / 2} 0 0"/>
         <geometry>
           <cylinder length="${height * scale}" radius="${radius * scale}"/>
@@ -45,10 +51,10 @@
         <parent link="${parent}" />
         <child link="${prefix}node2" />
-        <origin xyz="${x} ${y} ${z}" rpy="${R} ${P} ${Y + 3*pi/2}" />
+        <xacro:insert_block name="origin" />
     </joint>
     <joint name="${prefix}PMA3_joint" type="fixed">
         <parent link="${prefix}node2" />
         <child link="${prefix}PMA3" />
-        <origin xyz="0.100 0 -0.025" rpy="${pi/2} 0 0" />
+        <origin xyz="0 -0.1 -0.035" rpy="${pi/2} 0 ${-pi/2}" />
     </joint>
   </xacro:macro>

File: morpheus_description/urdf/macros/node2_table.xacro (robot description, xacro)
@@ -2,23 +2,36 @@
 <robot name="node2_table" xmlns:xacro="http://ros.org/wiki/xacro">
   <xacro:macro name="node2_table"
-      params="x:=0 y:=0 z:=0 R:=0 P:=0 Y:=0 scale:=1 prefix parent">
+    params="
+    prefix
+    parent
+    scale:=1
+    *origin">
     <xacro:include filename="$(find morpheus_description)/urdf/macros/hab_table.xacro" />
     <xacro:hab_table
-        prefix=""
-        parent="world"
-        x="${x}"
-        y="${y}"
-        z="${z}"
-        scale="1"
-    />
+      prefix=""
+      parent="world"
+      scale="1"
+    >
+      <xacro:insert_block name="origin" />
+    </xacro:hab_table>
     <xacro:include filename="$(find morpheus_description)/urdf/macros/node2.xacro" />
     <xacro:node2
-        prefix=""
-        parent="world"
-        x="${x + (0.0254 * 48)}"
-        y="${y + (0.0254 * 14.5)}"
-        z="${z + (0.0254 * 21)}"
-        scale="1"
-    />
+      prefix=""
+      parent="${prefix}hab_table"
+      scale="1"
+    >
+      <origin
+        xyz="
+          ${0.0254 * 48}
+          ${0.0254 * 14.5}
+          ${0.0254 * 21}
+        "
+        rpy="
+          0
+          0
+          0
+        "
+      />
+    </xacro:node2>
     <!-- scale=0.0254 meters/inch -->
   </xacro:macro>

File: morpheus_description/urdf/scenes/node2_dragon_scene.xacro (robot description, xacro)
@@ -2,21 +2,41 @@
 <robot xmlns:xacro="http://www.ros.org/wiki/xacro" name="node2_scene">
     <xacro:include filename="$(find morpheus_description)/urdf/macros/node2.xacro" />
-    <xacro:include filename="$(find morpheus_description)/urdf/macros/dragon_primitive.xacro" />
+    <xacro:include filename="$(find morpheus_description)/urdf/macros/dragon.xacro" />
     <xacro:node2
         prefix=""
         parent="world"
-        x="${0.0254 * 0}"
-        y="${0.0254 * (14.5 + 8.5)}"
-        z="${0.0254 * 21}"
         scale="1"
-    />
-    <xacro:dragon_primitive
+    >
+        <origin
+            xyz="
+                ${0.0254 * 0}
+                ${0.0254 * (14.5 + 8.5)}
+                ${0.0254 * 21}
+            "
+            rpy="
+                0
+                0
+                0
+            "
+        />
+    </xacro:node2>
+    <xacro:dragon
         prefix=""
         parent="world"
-        x="${0.0254 * 12}"
-        y="${0.0254 * 4}"
-        z="${0.0254 * 12}"
         scale="1"
-    />
+    >
+        <origin
+            xyz="
+                ${0.0254 * 12}
+                ${0.0254 * 20}
+                ${0.0254 * 32}
+            "
+            rpy="
+                0.5
+                -0.5
+                0.5
+            "
+        />
+    </xacro:dragon>
     <!-- scale=0.0254 meters/inch -->
 </robot>

File: morpheus_description/urdf/scenes/node2_scene.xacro (robot description, xacro)
@@ -5,9 +5,19 @@
         prefix=""
         parent="world"
-        x="${0.0254 * (-48)}"
-        y="${0.0254 * 8.5}"
-        z="${0.0254 * 34.75 * 0}"
         scale="1"
-    />
+    >
+        <origin
+            xyz="
+                ${0.0254 * (-48)}
+                ${0.0254 * 8.5}
+                ${0.0254 * 34.75 * 0}
+            "
+            rpy="
+                0
+                0
+                0
+            "
+        />
+    </xacro:node2_table>
     <!-- scale=0.0254 meters/inch -->
 </robot>
