Commit message: ROS2 Migration: Control revisions in progress. Cartesian controllers connect but behave unexpectedly. MoveIt control being ported as well to facilitate debugging.

File: morpheus_description/urdf/macros/ur_endeffector_macro.xacro (robot description, xacro)
@@ -1,4 +1,4 @@
 <?xml version="1.0"?>
-<robot xmlns:xacro="http://www.ros.org/wiki/xacro" name="b_bot">
+<robot xmlns:xacro="http://www.ros.org/wiki/xacro">
     <xacro:include filename="$(find ur_description)/urdf/ur_macro.xacro" />
     <xacro:include filename="$(find morpheus_description)/urdf/macros/d415_mount_macro.xacro" />
@@ -12,8 +12,8 @@
         *origin
         ur_type:='ur5e'
-        joint_limits_parameters_file:=$(find ur_description)/config/${ur_type}/joint_limits.yaml
-        kinematics_parameters_file:=$(find ur_description)/config/${ur_type}/default_kinematics.yaml
-        physical_parameters_file:=$(find ur_description)/config/${ur_type}/physical_parameters.yaml
-        visual_parameters_file:=$(find ur_description)/config/${ur_type}/visual_parameters.yaml
+        joint_limits_parameters_file:='$(find ur_description)/config/${ur_type}/joint_limits.yaml'
+        kinematics_parameters_file:='$(find ur_description)/config/${ur_type}/default_kinematics.yaml'
+        physical_parameters_file:='$(find ur_description)/config/${ur_type}/physical_parameters.yaml'
+        visual_parameters_file:='$(find ur_description)/config/${ur_type}/visual_parameters.yaml'
         safety_limits:=false
         safety_pos_margin:=0.15
@@ -22,6 +22,6 @@
         mount_type:='d415_mount'
         ee_type:=''
-        use_fake_hardware:=false
-        gazebo_sim:=false
+        use_mock_hardware:=false
+        sim_gazebo:=false
         device:=/dev/ttyUSB0
         sim_isaac:=false
@@ -55,69 +55,57 @@
             <xacro:insert_block name="origin" />
         </xacro:ur_robot>
-        <xacro:property name="last_link" value="wrist_3_link"/>
+        <xacro:property name="last_link" value="tool0"/>
         <!-- Mount for optional Realsense d415 camera -->
-        <xacro:choose>
-            <xacro:when value="${mount_type} == 'd415'">
-                <xacro:d415_mount
-                    prefix="${tf_prefix}"
-                    parent="${tf_prefix}${last_link}"
-                    >
-                    <origin xyz="0 0 0" rpy="0 0 0" />
-                </xacro:d415_mount>
-                <xacro:property name="last_link" value="d415_mount_attach_link"/>
-            </xacro:when>
-        </xacro:choose>
+        <xacro:if value="${mount_type == 'd415_mount'}">
+            <xacro:d415_mount
+                prefix="${tf_prefix}"
+                parent="${tf_prefix}${last_link}"
+                >
+                <origin xyz="0 0 0" rpy="0 0 ${pi}" />
+            </xacro:d415_mount>
+            <xacro:property name="last_link" value="d415_mount_attach_link"/>
+        </xacro:if>
         <!-- End Effector -->
-        <xacro:choose>
-            <xacro:when value="${ee_type} == 'robotiq'">
-                <xacro:ur_to_robotiq
-                    prefix="${tf_prefix}"
-                    parent="${tf_prefix}${last_link}"
-                    child="${tf_prefix}robotiq_2f_85_base_link"
-                    rotation="${pi}"
-                    >
-                </xacro:ur_to_robotiq>
-                <xacro:property name="last_link" value="d415_mount_attach_link"/>
-                <xacro:robotiq_gripper
-                    name="${tf_prefix}robotiq_2f_85"
-                    prefix="${tf_prefix}"
-                    parent="${tf_prefix}${last_link}"
-                    sim_gazebo="${sim_gazebo}"
-                    sim_isaac="${sim_isaac}"
-                    isaac_joint_commands="${isaac_joint_commands}"
-                    isaac_joint_states="${isaac_joint_states}"
-                    use_fake_hardware="${use_fake_hardware}"
-                    mock_sensor_commands="${mock_sensor_commands}"
-                    include_ros2_control="${include_ros2_control}"
-                    com_port="${device}"
-                    gripper_speed_multiplier="${gripper_speed_multiplier}"
-                    gripper_force_multiplier="${gripper_force_multiplier}"
-                    gripper_max_speed="${gripper_max_speed}"
-                    gripper_max_force="${gripper_max_force}"
-                    gripper_closed_position="${gripper_closed_position}"
-                    >
-                    <origin xyz="0 0 0.003" rpy="0 0 ${pi}" />
-                </xacro:robotiq_gripper>
-            </xacro:when>
-            <xacro:when value="${ee_type} == 'onrobot'">
-                <xacro:onrobot
-                    onrobot_type="rg2"
-                    prefix="${tf_prefix}"
-                    sim_gazebo="${sim_gazebo}"
-                    use_fake_hardware="${use_fake_hardware}"
-                    connection_type="${connection_type}"
-                    device="${device}"
-                    ip_address="${ip_address}"
-                    port="${port}"
-                    >
-                    <origin xyz="0 0 0.0026" rpy="0 0 ${pi}" />
-                </xacro:onrobot>
-                <joint name="${tf_prefix}onrobot_base_link_joint" type="fixed">
-                    <parent link="${tf_prefix}${last_link}"/>
-                    <child link="${tf_prefix}onrobot_base_link"/>
-                    <origin xyz="0 0 0" rpy="0 0 ${-pi/2}"/>
-                </joint>
-            </xacro:when>
-        </xacro:choose>
+        <xacro:if value="${ee_type == 'robotiq'}">
+            <xacro:robotiq_gripper
+                name="${tf_prefix}robotiq_2f_85"
+                prefix="${tf_prefix}"
+                parent="${tf_prefix}${last_link}"
+                sim_gazebo="${sim_gazebo}"
+                sim_isaac="${sim_isaac}"
+                isaac_joint_commands="${isaac_joint_commands}"
+                isaac_joint_states="${isaac_joint_states}"
+                use_fake_hardware="${use_mock_hardware}"
+                mock_sensor_commands="${mock_sensor_commands}"
+                include_ros2_control="${include_ros2_control}"
+                com_port="${device}"
+                gripper_speed_multiplier="${gripper_speed_multiplier}"
+                gripper_force_multiplier="${gripper_force_multiplier}"
+                gripper_max_speed="${gripper_max_speed}"
+                gripper_max_force="${gripper_max_force}"
+                gripper_closed_position="${gripper_closed_position}"
+                >
+                <origin xyz="0 0 0.003" rpy="0 0 0" />
+            </xacro:robotiq_gripper>
+        </xacro:if>
+        <xacro:if value="${ee_type == 'onrobot'}">
+            <xacro:onrobot
+                onrobot_type="rg2"
+                prefix="${tf_prefix}"
+                sim_gazebo="${sim_gazebo}"
+                use_fake_hardware="${use_mock_hardware}"
+                connection_type="${connection_type}"
+                device="${device}"
+                ip_address="${ip_address}"
+                port="${port}"
+                >
+                <origin xyz="0 0 0.0026" rpy="0 0 0" />
+            </xacro:onrobot>
+            <joint name="${tf_prefix}onrobot_base_link_joint" type="fixed">
+                <parent link="${tf_prefix}${last_link}"/>
+                <child link="${tf_prefix}onrobot_base_link"/>
+                <origin xyz="0 0 0" rpy="0 0 ${-pi/2}"/>
+            </joint>
+        </xacro:if>
     </xacro:macro>
 </robot>

File: morpheus_description/urdf/scenes/ur_endeffector.urdf.xacro (robot description, xacro)
@@ -20,5 +20,5 @@
     <xacro:arg name="ee_type" default="robotiq"/>
     <!-- Common End Effector Arguments -->
-    <xacro:arg name="use_fake_hardware" default="false"/>
+    <xacro:arg name="use_mock_hardware" default="false"/>
     <xacro:arg name="sim_gazebo" default="false"/>
     <xacro:arg name="device" default="/dev/ttyUSB0"/>
@@ -30,8 +30,8 @@
     <xacro:arg name="include_ros2_control" default="true"/>
     <xacro:arg name="gripper_speed_multiplier" default="1.0"/>
-    <xacro:arg name="gripper_speed_multiplier" default="0.5"/>
-    <xacro:arg name="gripper_speed_multiplier" default="0.150"/>
-    <xacro:arg name="gripper_speed_multiplier" default="235.0"/>
-    <xacro:arg name="gripper_speed_multiplier" default="0.7929"/>
+    <xacro:arg name="gripper_force_multiplier" default="0.5"/>
+    <xacro:arg name="gripper_max_speed" default="0.150"/>
+    <xacro:arg name="gripper_max_force" default="235.0"/>
+    <xacro:arg name="gripper_closed_position" default="0.7929"/>
     <!-- OnRobot Gripper Arguments -->
     <xacro:arg name="connection_type" default="serial"/>
@@ -39,11 +39,8 @@
     <xacro:arg name="port" default="502"/>
     <!-- Additional URDF Files -->
-    <xacro:arg name="environment_file" default="$(find morpheus_description)/urdf/scenes/node2.urdf.xacro"/>
+    <xacro:arg name="environment_file" default=""/>
     <link name="world"/>
     <!-- Includes -->
     <xacro:include filename="$(find morpheus_description)/urdf/macros/ur_endeffector_macro.xacro" />
-    <xacro:if value="$(arg environment_file) != ''">
-        <xacro:include filename="$(arg environment_file)"/>
-    </xacro:if>
     <!-- Robot -->
     <xacro:ur_endeffector
@@ -62,7 +59,7 @@
         mount_type="$(arg mount_type)"
         ee_type="$(arg ee_type)"
-        use_fake_hardware="$(arg use_fake_hardware)"
+        use_mock_hardware="$(arg use_mock_hardware)"
         sim_gazebo="$(arg sim_gazebo)"
-        device="$(arg /dev/device)"
+        device="$(arg device)"
         sim_isaac="$(arg sim_isaac)"
         isaac_joint_commands="$(arg isaac_joint_commands)"
@@ -70,5 +67,4 @@
         mock_sensor_commands="$(arg mock_sensor_commands)"
         include_ros2_control="$(arg include_ros2_control)"
-        com_port="$(arg device)"
         gripper_speed_multiplier="$(arg gripper_speed_multiplier)"
         gripper_force_multiplier="$(arg gripper_force_multiplier)"
@@ -82,13 +78,7 @@
         <origin xyz="0 0 0" rpy="0 0 0" />          <!-- position robot in the world -->
     </xacro:ur_endeffector>
-    <!-- Environment -->
-    <xacro:node2_table
-        prefix="$(arg tf_prefix)"
-        parent="world"
-        x="${0.0254 * (-48)}"
-        y="${0.0254 * 8.5}"
-        z="${0.0254 * 34.75}"
-        scale="1"
-    />
-    <!-- scale=0.0254 meters/inch -->
+    <!-- Create the environment around the robot -->
+    <xacro:if value="${environment_file}">
+        <xacro:include filename="$(arg environment_file)"/>
+    </xacro:if>
 </robot>

File: morpheus_driver/urdf/ur_control.urdf.xacro (robot description, xacro)
@@ -46,5 +46,5 @@
     <xacro:property name="initial_positions_file" default="$(arg initial_positions_file)"/>
     <!-- Additional URDF Files -->
-    <xacro:arg name="environment_file" default="$(find morpheus_description)/urdf/scenes/node2.urdf.xacro"/>
+    <xacro:arg name="environment_file" default=""/>
     <!-- UR Robot Include -->
     <xacro:include filename="$(find ur_description)/urdf/ur_macro.xacro"/>
@@ -99,4 +99,6 @@
     />
     <!-- Create the environment around the robot -->
-    <xacro:include filename="$(arg environment_file)"/>
+    <xacro:if value="${arg environment_file}">
+        <xacro:include filename="$(arg environment_file)"/>
+    </xacro:if>
 </robot>

File: morpheus_driver/urdf/ur_endeffector_control.urdf.xacro (robot description, xacro)
@@ -18,9 +18,9 @@
     <!-- ros2_control Parameters -->
     <xacro:arg name="headless_mode" default="false" />
-    <xacro:arg name="robot_ip" default="0.0.0.0"/>
+    <xacro:arg name="robot_ip" default="192.168.1.102"/>
     <xacro:arg name="ur_script_filename" default="$(find ur_client_library)/resources/external_control.urscript"/>
     <xacro:arg name="ur_output_recipe_filename" default="$(find ur_robot_driver)/resources/rtde_output_recipe.txt"/>
     <xacro:arg name="ur_input_recipe_filename" default="$(find ur_robot_driver)/resources/rtde_input_recipe.txt"/>
-    <xacro:arg name="reverse_ip" default="0.0.0.0"/>
+    <xacro:arg name="reverse_ip" default="192.168.1.2"/>
     <xacro:arg name="script_command_port" default="50004"/>
     <xacro:arg name="reverse_port" default="50001"/>
@@ -28,5 +28,5 @@
     <xacro:arg name="trajectory_port" default="50003"/>
     <!-- Tool Communication Parameters-->
-    <xacro:arg name="use_tool_communication" default="false" />
+    <xacro:arg name="use_tool_communication" default="true" />
     <xacro:arg name="tool_voltage" default="0" />
     <xacro:arg name="tool_parity" default="0" />
@@ -38,6 +38,6 @@
     <xacro:arg name="tool_tcp_port" default="54321" />
     <!-- Simulation Parameters -->
-    <xacro:arg name="use_mock_hardware" default="false" />
-    <xacro:arg name="mock_sensor_commands" default="false" />
+    <xacro:arg name="use_mock_hardware" default="true" />
+    <xacro:arg name="mock_sensor_commands" default="true" />
     <xacro:arg name="simulation_controllers" default="$(find morpheus_sim)/config/ur/ur5e/ur_controllers.yaml" />
     <!-- Initial position for simulations (Mock Hardware, Gazebo, Ignition) -->
@@ -50,18 +50,16 @@
     <xacro:arg name="ee_type" default="robotiq"/>
     <!-- Common End Effector Arguments -->
-    <xacro:arg name="use_fake_hardware" default="false"/>
     <xacro:arg name="sim_gazebo" default="false"/>
-    <xacro:arg name="device" default="/dev/ttyUSB0"/>
+    <xacro:arg name="device" default="/tmp/ttyUR"/>
     <!-- Robotiq Gripper Arguments -->
     <xacro:arg name="sim_isaac" default="false"/>
     <xacro:arg name="isaac_joint_commands" default="/isaac_joint_commands"/>
     <xacro:arg name="isaac_joint_states" default="/isaac_joint_states"/>
-    <xacro:arg name="mock_sensor_commands" default="false"/>
     <xacro:arg name="include_ros2_control" default="true"/>
     <xacro:arg name="gripper_speed_multiplier" default="1.0"/>
-    <xacro:arg name="gripper_speed_multiplier" default="0.5"/>
-    <xacro:arg name="gripper_speed_multiplier" default="0.150"/>
-    <xacro:arg name="gripper_speed_multiplier" default="235.0"/>
-    <xacro:arg name="gripper_speed_multiplier" default="0.7929"/>
+    <xacro:arg name="gripper_force_multiplier" default="0.5"/>
+    <xacro:arg name="gripper_max_speed" default="0.150"/>
+    <xacro:arg name="gripper_max_force" default="235.0"/>
+    <xacro:arg name="gripper_closed_position" default="0.7929"/>
     <!-- OnRobot Gripper Arguments -->
     <xacro:arg name="connection_type" default="serial"/>
@@ -69,5 +67,5 @@
     <xacro:arg name="port" default="502"/>
     <!-- Additional URDF Files -->
-    <xacro:arg name="environment_file" default="$(find morpheus_description)/urdf/scenes/node2.urdf.xacro" />
+    <xacro:arg name="environment_file" default="" />
     <!-- Robot Include -->
     <xacro:include filename="$(find morpheus_description)/urdf/macros/ur_endeffector_macro.xacro" />
@@ -92,7 +90,7 @@
         mount_type="$(arg mount_type)"
         ee_type="$(arg ee_type)"
-        use_fake_hardware="$(arg use_fake_hardware)"
+        use_mock_hardware="$(arg use_mock_hardware)"
         sim_gazebo="$(arg sim_gazebo)"
-        device="$(arg /dev/device)"
+        device="$(arg device)"
         sim_isaac="$(arg sim_isaac)"
         isaac_joint_commands="$(arg isaac_joint_commands)"
@@ -100,5 +98,4 @@
         mock_sensor_commands="$(arg mock_sensor_commands)"
         include_ros2_control="$(arg include_ros2_control)"
-        com_port="$(arg device)"
         gripper_speed_multiplier="$(arg gripper_speed_multiplier)"
         gripper_force_multiplier="$(arg gripper_force_multiplier)"
@@ -142,4 +139,7 @@
     />
     <!-- Create the environment around the robot -->
-    <xacro:include filename="$(arg environment_file)"/>
+    <xacro:property name="environment_file" value="$(arg environment_file)"/>
+    <xacro:if value="${environment_file != ''}">
+        <xacro:include filename="$(arg environment_file)"/>
+    </xacro:if>
 </robot>

Commit message: OnRobot gripper integration in progress

File: morpheus_description/urdf/macros/ur_endeffector_macro.xacro (robot description, xacro)
@@ -91,4 +91,5 @@
         <xacro:if value="${ee_type == 'onrobot'}">
             <xacro:onrobot
+                name="${tf_prefix}onrobot_rg2"
                 onrobot_type="rg2"
                 prefix="${tf_prefix}"
@@ -100,10 +101,9 @@
                 port="${port}"
                 >
-                <origin xyz="0 0 0.0026" rpy="0 0 0" />
             </xacro:onrobot>
             <joint name="${tf_prefix}onrobot_base_link_joint" type="fixed">
                 <parent link="${tf_prefix}${last_link}"/>
                 <child link="${tf_prefix}onrobot_base_link"/>
-                <origin xyz="0 0 0" rpy="0 0 ${-pi/2}"/>
+                <origin xyz="0 0 0.0026" rpy="0 0 ${-pi/2}"/>
             </joint>
         </xacro:if>
