Commit message: Proximity marker position bug fix, teleop build tweaks to ensure executables show up correctly

File: morpheus_description/urdf/scenes/ur_endeffector.urdf.xacro (robot description, xacro)
@@ -79,5 +79,6 @@
     </xacro:ur_endeffector>
     <!-- Create the environment around the robot -->
-    <xacro:if value="${environment_file}">
+    <xacro:property name="environment_file" value="$(arg environment_file)"/>
+    <xacro:if value="${environment_file != ''}">
         <xacro:include filename="$(arg environment_file)"/>
     </xacro:if>
