Commit message: Moveit srdf and launch improvements to better accomodate onrobot grippers. Teleop build tweaks to fix the includes

File: morpheus_description/srdf/macros/ur_onrobot_macro.srdf.xacro (robot description, xacro)
@@ -15,13 +15,13 @@
         </group>
         <group name="gripper">
-            <joint name="quick_changer_joint"/>
-            <joint name="angle_bracket_joint"/>
-            <joint name="gripper_body_joint"/>
             <joint name="finger_joint"/>
+            <joint name="finger_width"/>
             <joint name="right_inner_finger_joint"/>
             <joint name="left_inner_knuckle_joint"/>
-            <joint name="left_outer_knuckle_joint"/>
+            <joint name="right_outer_knuckle_joint"/>
             <joint name="left_inner_finger_joint"/>
             <joint name="right_inner_knuckle_joint"/>
+            <joint name="left_finger_tip_joint"/>
+            <joint name="right_finger_tip_joint"/>
         </group>
         <!--GROUP STATES: Purpose: Define a named state for a particular group, in terms of joint values. This is useful to define states like 'folded arms'-->
@@ -44,9 +44,9 @@
         <group_state name="open" group="gripper">
             <joint name="finger_joint" value="0"/>
-            <joint name="left_outer_knuckle_joint" value="0"/>
+            <joint name="right_outer_knuckle_joint" value="0"/>
         </group_state>
         <group_state name="close" group="gripper">
             <joint name="finger_joint" value="1.18"/>
-            <joint name="left_outer_knuckle_joint" value="1.18"/>
+            <joint name="right_outer_knuckle_joint" value="1.18"/>
         </group_state>
         <!--END EFFECTOR: Purpose: Represent information about an end effector.-->
@@ -59,26 +59,13 @@
         <passive_joint name="left_inner_finger_joint"/>
         <passive_joint name="right_inner_knuckle_joint"/>
+        <passive_joint name="left_finger_tip_joint"/>
+        <passive_joint name="right_finger_tip_joint"/>
         <!--DISABLE COLLISIONS: By default it is assumed that any link of the robot could potentially come into collision with any other link in the robot. This tag disables collision checking between a specified pair of links. -->
-        <disable_collisions link1="angle_bracket" link2="camera_link" reason="Never"/>
-        <disable_collisions link1="angle_bracket" link2="d415_mount_link" reason="Never"/>
-        <disable_collisions link1="angle_bracket" link2="gripper_body" reason="Adjacent"/>
-        <disable_collisions link1="angle_bracket" link2="left_inner_finger" reason="Never"/>
-        <disable_collisions link1="angle_bracket" link2="left_inner_knuckle" reason="Never"/>
-        <disable_collisions link1="angle_bracket" link2="left_outer_knuckle" reason="Never"/>
-        <disable_collisions link1="angle_bracket" link2="quick_changer" reason="Adjacent"/>
-        <disable_collisions link1="angle_bracket" link2="right_inner_finger" reason="Never"/>
-        <disable_collisions link1="angle_bracket" link2="right_inner_knuckle" reason="Never"/>
-        <disable_collisions link1="angle_bracket" link2="right_outer_knuckle" reason="Never"/>
-        <disable_collisions link1="angle_bracket" link2="wrist_1_link" reason="Never"/>
-        <disable_collisions link1="angle_bracket" link2="wrist_2_link" reason="Never"/>
-        <disable_collisions link1="angle_bracket" link2="wrist_3_link" reason="Never"/>
-        <disable_collisions link1="base_link_inertia" link2="pedestal" reason="Adjacent"/>
         <disable_collisions link1="base_link_inertia" link2="shoulder_link" reason="Adjacent"/>
         <disable_collisions link1="camera_link" link2="d415_mount_link" reason="Adjacent"/>
-        <disable_collisions link1="camera_link" link2="gripper_body" reason="Never"/>
+        <disable_collisions link1="camera_link" link2="onrobot_base_link" reason="Never"/>
         <disable_collisions link1="camera_link" link2="left_inner_finger" reason="Never"/>
         <disable_collisions link1="camera_link" link2="left_inner_knuckle" reason="Never"/>
         <disable_collisions link1="camera_link" link2="left_outer_knuckle" reason="Never"/>
-        <disable_collisions link1="camera_link" link2="quick_changer" reason="Never"/>
         <disable_collisions link1="camera_link" link2="right_inner_finger" reason="Never"/>
         <disable_collisions link1="camera_link" link2="right_inner_knuckle" reason="Never"/>
@@ -87,9 +74,8 @@
         <disable_collisions link1="camera_link" link2="wrist_2_link" reason="Never"/>
         <disable_collisions link1="camera_link" link2="wrist_3_link" reason="Never"/>
-        <disable_collisions link1="d415_mount_link" link2="gripper_body" reason="Never"/>
+        <disable_collisions link1="d415_mount_link" link2="onrobot_base_link" reason="Never"/>
         <disable_collisions link1="d415_mount_link" link2="left_inner_finger" reason="Never"/>
         <disable_collisions link1="d415_mount_link" link2="left_inner_knuckle" reason="Never"/>
         <disable_collisions link1="d415_mount_link" link2="left_outer_knuckle" reason="Never"/>
-        <disable_collisions link1="d415_mount_link" link2="quick_changer" reason="Adjacent"/>
         <disable_collisions link1="d415_mount_link" link2="right_inner_finger" reason="Never"/>
         <disable_collisions link1="d415_mount_link" link2="right_inner_knuckle" reason="Never"/>
@@ -101,17 +87,15 @@
         <disable_collisions link1="forearm_link" link2="wrist_1_link" reason="Adjacent"/>
         <disable_collisions link1="forearm_link" link2="wrist_2_link" reason="Never"/>
-        <disable_collisions link1="gripper_body" link2="left_inner_finger" reason="Never"/>
-        <disable_collisions link1="gripper_body" link2="left_inner_knuckle" reason="Adjacent"/>
-        <disable_collisions link1="gripper_body" link2="left_outer_knuckle" reason="Adjacent"/>
-        <disable_collisions link1="gripper_body" link2="quick_changer" reason="Never"/>
-        <disable_collisions link1="gripper_body" link2="right_inner_finger" reason="Never"/>
-        <disable_collisions link1="gripper_body" link2="right_inner_knuckle" reason="Adjacent"/>
-        <disable_collisions link1="gripper_body" link2="right_outer_knuckle" reason="Adjacent"/>
-        <disable_collisions link1="gripper_body" link2="wrist_1_link" reason="Never"/>
-        <disable_collisions link1="gripper_body" link2="wrist_2_link" reason="Never"/>
-        <disable_collisions link1="gripper_body" link2="wrist_3_link" reason="Never"/>
+        <disable_collisions link1="onrobot_base_link" link2="left_inner_finger" reason="Never"/>
+        <disable_collisions link1="onrobot_base_link" link2="left_inner_knuckle" reason="Adjacent"/>
+        <disable_collisions link1="onrobot_base_link" link2="left_outer_knuckle" reason="Adjacent"/>
+        <disable_collisions link1="onrobot_base_link" link2="right_inner_finger" reason="Never"/>
+        <disable_collisions link1="onrobot_base_link" link2="right_inner_knuckle" reason="Adjacent"/>
+        <disable_collisions link1="onrobot_base_link" link2="right_outer_knuckle" reason="Adjacent"/>
+        <disable_collisions link1="onrobot_base_link" link2="wrist_1_link" reason="Never"/>
+        <disable_collisions link1="onrobot_base_link" link2="wrist_2_link" reason="Never"/>
+        <disable_collisions link1="onrobot_base_link" link2="wrist_3_link" reason="Never"/>
         <disable_collisions link1="left_inner_finger" link2="left_inner_knuckle" reason="Default"/>
         <disable_collisions link1="left_inner_finger" link2="left_outer_knuckle" reason="Adjacent"/>
-        <disable_collisions link1="left_inner_finger" link2="quick_changer" reason="Never"/>
         <disable_collisions link1="left_inner_finger" link2="right_inner_finger" reason="Never"/>
         <disable_collisions link1="left_inner_finger" link2="right_inner_knuckle" reason="Never"/>
@@ -121,5 +105,4 @@
         <disable_collisions link1="left_inner_finger" link2="wrist_3_link" reason="Never"/>
         <disable_collisions link1="left_inner_knuckle" link2="left_outer_knuckle" reason="Default"/>
-        <disable_collisions link1="left_inner_knuckle" link2="quick_changer" reason="Never"/>
         <disable_collisions link1="left_inner_knuckle" link2="right_inner_finger" reason="Never"/>
         <disable_collisions link1="left_inner_knuckle" link2="right_inner_knuckle" reason="Never"/>
@@ -128,5 +111,4 @@
         <disable_collisions link1="left_inner_knuckle" link2="wrist_2_link" reason="Never"/>
         <disable_collisions link1="left_inner_knuckle" link2="wrist_3_link" reason="Never"/>
-        <disable_collisions link1="left_outer_knuckle" link2="quick_changer" reason="Never"/>
         <disable_collisions link1="left_outer_knuckle" link2="right_inner_finger" reason="Never"/>
         <disable_collisions link1="left_outer_knuckle" link2="right_inner_knuckle" reason="Never"/>
@@ -135,11 +117,4 @@
         <disable_collisions link1="left_outer_knuckle" link2="wrist_2_link" reason="Never"/>
         <disable_collisions link1="left_outer_knuckle" link2="wrist_3_link" reason="Never"/>
-        <disable_collisions link1="pedestal" link2="shoulder_link" reason="Never"/>
-        <disable_collisions link1="quick_changer" link2="right_inner_finger" reason="Never"/>
-        <disable_collisions link1="quick_changer" link2="right_inner_knuckle" reason="Never"/>
-        <disable_collisions link1="quick_changer" link2="right_outer_knuckle" reason="Never"/>
-        <disable_collisions link1="quick_changer" link2="wrist_1_link" reason="Never"/>
-        <disable_collisions link1="quick_changer" link2="wrist_2_link" reason="Never"/>
-        <disable_collisions link1="quick_changer" link2="wrist_3_link" reason="Never"/>
         <disable_collisions link1="right_inner_finger" link2="right_inner_knuckle" reason="Default"/>
         <disable_collisions link1="right_inner_finger" link2="right_outer_knuckle" reason="Adjacent"/>
